File: eagle/lightdimmer_rc.brd (EAGLE design)
At the start: 102.8 x 26.3 mm, 14 parts, among them Q1 IPA040N06N, T1 BC238

Commit message: Updated to actual version
Parts:
- added R4: 2K2, rcl:0204/7
- moved R3 8.98 mm to (16.5, 21.6), turned to 90 degrees
- moved T1 2.84 mm to (20.3, 17.8), turned to 270 degrees
Connections:
- net N$10: now also R4.1
- net N$3: now also R4.2
Routing:
- net N$3: track 76.7 -> 108.3 mm
- net N$10: track 65.8 -> 85.7 mm
- net N$8: track 11.2 -> 20.8 mm
- net N$7: track 37.2 -> 33.9 mm
Changed lines of the file:
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@@
 <element name="U$2" library="433mhz" package="RECV433MHZ" value="RECV433MHZ" x="92.71" y="5.08"/>
 <element name="U$3" library="LM2596_DCDC" package="LM2596DCDC" value="LM2596DCDC" x="45.72" y="12.7"/>
-<element name="T1" library="transistor" package="TO92-CBE" value="BC238" x="17.78" y="19.05"/>
+<element name="T1" library="transistor" package="TO92-CBE" value="BC238" x="20.32" y="17.78" rot="R270"/>
 <element name="R2" library="rcl" package="0204/7" value="560" x="12.7" y="15.24" rot="R180"/>
-<element name="R3" library="rcl" package="0204/7" value="10K" x="22.86" y="15.24"/>
+<element name="R3" library="rcl" package="0204/7" value="10K" x="16.51" y="21.59" rot="R90"/>
+<element name="R4" library="rcl" package="0204/7" value="2K2" x="33.02" y="24.13"/>
 </elements>
 <signals>
@@
 <contactref element="C1" pad="1"/>
 <wire x1="64.525" y1="20.52" x2="64.97" y2="20.52" width="1.27" layer="16"/>
-<wire x1="64.97" y1="20.52" x2="68.58" y2="24.13" width="1.27" layer="16"/>
-<wire x1="68.58" y1="24.13" x2="82.55" y2="24.13" width="1.27" layer="16"/>
+<wire x1="68.58" y1="24.13" x2="69.85" y2="24.13" width="1.27" layer="16"/>
+<wire x1="69.85" y1="24.13" x2="82.55" y2="24.13" width="1.27" layer="16"/>
 <wire x1="82.55" y1="24.13" x2="95.25" y2="24.13" width="1.27" layer="16"/>
 <wire x1="95.25" y1="24.13" x2="95.25" y2="22.2875" width="1.27" layer="16"/>
@@
 <wire x1="96.52" y1="10.16" x2="97.79" y2="11.43" width="1.016" layer="16"/>
 <wire x1="97.79" y1="11.43" x2="97.79" y2="13.97" width="1.016" layer="16"/>
+<contactref element="R4" pad="2"/>
+<wire x1="69.85" y1="24.13" x2="64.77" y2="24.13" width="1.27" layer="16"/>
+<wire x1="64.77" y1="24.13" x2="36.83" y2="24.13" width="1.016" layer="16"/>
+<wire x1="64.97" y1="20.52" x2="64.97" y2="23.93" width="1.27" layer="16"/>
+<wire x1="64.97" y1="23.93" x2="64.77" y2="24.13" width="1.016" layer="16"/>
 </signal>
 <signal name="N$4">
@@
 <contactref element="+12V" pad="P$1"/>
 <contactref element="R2" pad="2"/>
-<wire x1="24.49" y1="20.52" x2="22.15" y2="22.86" width="1.6764" layer="16"/>
-<wire x1="22.15" y1="22.86" x2="11.43" y2="22.86" width="1.6764" layer="16"/>
-<wire x1="11.43" y1="22.86" x2="10.16" y2="21.59" width="1.6764" layer="16"/>
+<wire x1="24.49" y1="20.52" x2="22.15" y2="22.86" width="1.27" layer="16"/>
+<wire x1="22.15" y1="22.86" x2="11.43" y2="22.86" width="1.27" layer="16"/>
+<wire x1="11.43" y1="22.86" x2="10.16" y2="21.59" width="1.27" layer="16"/>
 <wire x1="6.35" y1="21.59" x2="10.16" y2="21.59" width="2.54" layer="16"/>
 <wire x1="3.81" y1="21.59" x2="6.35" y2="21.59" width="2.54" layer="16"/>
@@
 <contactref element="R3" pad="2"/>
 <wire x1="91.9975" y1="16.495" x2="27.925" y2="16.495" width="1.016" layer="16"/>
-<wire x1="27.925" y1="16.495" x2="26.67" y2="15.24" width="1.016" layer="16"/>
+<contactref element="R4" pad="1"/>
+<wire x1="27.925" y1="25.385" x2="27.925" y2="24.13" width="1.016" layer="16"/>
+<wire x1="27.925" y1="24.13" x2="27.925" y2="16.495" width="1.016" layer="16"/>
+<wire x1="29.21" y1="24.13" x2="27.925" y2="24.13" width="1.016" layer="16"/>
+<wire x1="16.51" y1="25.4" x2="27.91" y2="25.4" width="1.016" layer="16"/>
+<wire x1="27.91" y1="25.4" x2="27.925" y2="25.385" width="1.016" layer="16"/>
 </signal>
 <signal name="N$11">
@@
 <wire x1="3.81" y1="2.54" x2="16.51" y2="2.54" width="2.54" layer="16"/>
 <wire x1="16.51" y1="2.54" x2="17.78" y2="3.81" width="1.6764" layer="16"/>
-<wire x1="24.49" y1="3.345" x2="24.025" y2="3.81" width="1.6764" layer="16"/>
-<wire x1="24.025" y1="3.81" x2="21.59" y2="3.81" width="1.6764" layer="16"/>
-<wire x1="17.78" y1="3.81" x2="21.59" y2="3.81" width="1.6764" layer="16"/>
-<wire x1="21.59" y1="3.81" x2="21.59" y2="17.78" width="1.016" layer="16"/>
-<wire x1="21.59" y1="17.78" x2="20.32" y2="19.05" width="1.016" layer="16"/>
+<wire x1="24.49" y1="3.345" x2="24.025" y2="3.81" width="1.27" layer="16"/>
+<wire x1="17.78" y1="3.81" x2="22.86" y2="3.81" width="1.27" layer="16"/>
+<wire x1="22.86" y1="3.81" x2="24.025" y2="3.81" width="1.27" layer="16"/>
+<wire x1="20.32" y1="15.24" x2="22.86" y2="12.7" width="1.016" layer="16"/>
+<wire x1="22.86" y1="12.7" x2="22.86" y2="3.81" width="1.016" layer="16"/>
 </signal>
 <signal name="N$8">
@@
 <contactref element="R2" pad="1"/>
 <contactref element="Q1" pad="G"/>
-<wire x1="16.51" y1="15.24" x2="15.24" y2="16.51" width="1.016" layer="16"/>
-<wire x1="15.24" y1="16.51" x2="15.24" y2="19.05" width="1.016" layer="16"/>
 <wire x1="17.78" y1="8.89" x2="16.51" y2="10.16" width="1.016" layer="16"/>
 <wire x1="16.51" y1="10.16" x2="16.51" y2="15.24" width="1.016" layer="16"/>
+<wire x1="20.32" y1="20.32" x2="13.97" y2="20.32" width="1.016" layer="16"/>
+<wire x1="13.97" y1="20.32" x2="13.97" y2="15.24" width="1.016" layer="16"/>
+<wire x1="13.97" y1="15.24" x2="16.51" y2="15.24" width="1.016" layer="16"/>
 </signal>
 <signal name="N$12">
 <contactref element="R3" pad="1"/>
 <contactref element="T1" pad="B"/>
-<wire x1="19.05" y1="15.24" x2="17.78" y2="19.05" width="1.016" layer="16"/>
+<wire x1="16.51" y1="17.78" x2="20.32" y2="17.78" width="1.016" layer="16"/>
 </signal>
 </signals>
