File: eagle/lightdimmer_rc.sch (EAGLE design)
At the start: 14 parts, among them Q1 IPA040N06N, T1 BC238

Commit message: Updated to actual version
Parts:
- added R4: 2K2, rcl:R-EU_0204/7
Connections:
- net N$10: now also R4.1
- net N$3: now also R4.2
Changed lines of the file:
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@@
 <part name="R2" library="rcl" deviceset="R-EU_" device="0204/7" value="560"/>
 <part name="R3" library="rcl" deviceset="R-EU_" device="0204/7" value="10K"/>
+<part name="R4" library="rcl" deviceset="R-EU_" device="0204/7" value="2K2"/>
 </parts>
 <sheets>
@@
 <instance part="R2" gate="G$1" x="53.34" y="50.8" rot="R90"/>
 <instance part="R3" gate="G$1" x="81.28" y="63.5"/>
+<instance part="R4" gate="G$1" x="106.68" y="91.44" rot="R90"/>
 </instances>
 <busses>
@@
 <wire x1="55.88" y1="83.82" x2="68.58" y2="83.82" width="0.1524" layer="91"/>
 <wire x1="114.3" y1="86.36" x2="111.76" y2="86.36" width="0.1524" layer="91"/>
-<wire x1="111.76" y1="86.36" x2="111.76" y2="91.44" width="0.1524" layer="91"/>
-<wire x1="111.76" y1="91.44" x2="55.88" y2="91.44" width="0.1524" layer="91"/>
-<wire x1="55.88" y1="91.44" x2="55.88" y2="83.82" width="0.1524" layer="91"/>
+<wire x1="111.76" y1="86.36" x2="111.76" y2="99.06" width="0.1524" layer="91"/>
+<wire x1="111.76" y1="99.06" x2="106.68" y2="99.06" width="0.1524" layer="91"/>
+<wire x1="106.68" y1="99.06" x2="55.88" y2="99.06" width="0.1524" layer="91"/>
+<wire x1="55.88" y1="99.06" x2="55.88" y2="83.82" width="0.1524" layer="91"/>
 <junction x="55.88" y="83.82"/>
 <pinref part="R1" gate="G$1" pin="1"/>
@@
 <wire x1="55.88" y1="76.2" x2="55.88" y2="78.74" width="0.1524" layer="91"/>
 <junction x="55.88" y="78.74"/>
+<pinref part="R4" gate="G$1" pin="2"/>
+<wire x1="106.68" y1="96.52" x2="106.68" y2="99.06" width="0.1524" layer="91"/>
+<junction x="106.68" y="99.06"/>
 </segment>
 </net>
@@
 <pinref part="R3" gate="G$1" pin="2"/>
 <wire x1="106.68" y1="63.5" x2="86.36" y2="63.5" width="0.1524" layer="91"/>
+<pinref part="R4" gate="G$1" pin="1"/>
+<wire x1="106.68" y1="78.74" x2="106.68" y2="86.36" width="0.1524" layer="91"/>
+<junction x="106.68" y="78.74"/>
 </segment>
 </net>
